File: actuation.kicad_pcb (KiCad board)
At the start: 4 copper layers, 269 parts, among them J1 ACTUATION, J10 ACT CH9, J11 ACT CH10, J12 ACT CH11, J13 ACT CH12, J14 ACT CH13, J15 ACT CH14, J16 ACT CH15, J17 ACT CH16, J18 FB CH1, J19 FB CH2, J2 ACT CH1, J20 FB CH3, J21 FB CH4, J22 VDET CH1, J23 VDET CH2, J24 PWR IN, J25 PWR PROT, J26 PWR 3.3V, J27 SAFING, J28 ARM, J29 ACT HOT, J3 ACT CH2, J30 ACT COLD, J4 ACT CH3, J5 ACT CH4, J6 ACT CH5, J7 ACT CH6, J8 ACT CH7, J9 ACT CH8, K1 J115F11C, Q1 SI7220 NMOS, Q2 NMOS, U1 TPD4E02B04DQA, U10 TLP241A, U11 TLP241A, U12 TLP241A, U13 TLP241A, U14 TLP241A, U15 TLP241A, U16 TLP241A, U17 TLP241A, U18 TLP241A, U19 PCA9534, U2 PCA9615, U20 PCA9534, U21 OPTO_TLP2366_V4-TPL,E, U22 OPTO_TLP2366_V4-TPL,E, U23 OPTO_TLP2366_V4-TPL,E, U24 OPTO_TLP2366_V4-TPL,E, U25 OPTO_TLP2366_V4-TPL,E, U26 OPTO_TLP2366_V4-TPL,E, U27 TLV7031, U28 TLV7031, U29 OPTO_TLP2366_V4-TPL,E, U3 TLP241A, U30 OPTO_TLP2366_V4-TPL,E, U31 74LVC1G126, U32 PCA9534, U33 SN74LVC541A, U34 TLI4971, U35 LTC4367, U36 ADS1110, U37 AP64350, U38 TLP241A, U39 LP5912-3.3DRV, U4 TLP241A, U5 TLP241A, U6 TLP241A, U7 TLP241A, U8 TLP241A, U9 TLP241A

Commit message: Experimentation with placement
Parts:
- moved J27 326.6 mm to (319.6, -39.8), turned to 90 degrees
- moved U34 303.6 mm to (311.6, -54.9), turned to -90 degrees
- moved J24 302.1 mm to (320.7, -70.3), turned to 90 degrees
- moved J10 294.9 mm to (278.6, -93.3), turned to 180 degrees
- moved K1 294.0 mm to (292.1, -53.7), turned to 180 degrees
- moved J11 267.9 mm to (266.6, -93.3), turned to 180 degrees
- moved U10 240.7 mm to (277.9, -27.4), turned to -90 degrees
- moved J12 238.9 mm to (254.6, -93.3), turned to 180 degrees
- moved J14 233.0 mm to (230.6, -93.3), turned to 180 degrees
- moved J8 230.3 mm to (265.7, -13.0)
- moved J9 217.1 mm to (277.7, -13.0)
- moved J15 215.3 mm to (218.6, -93.3), turned to 180 degrees
- moved D10 192.2 mm to (277.8, -19.7)
- moved J16 186.3 mm to (206.6, -93.3), turned to 180 degrees
- moved J13 184.4 mm to (242.6, -93.3), turned to 180 degrees
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
Commit message: More placement
Parts:
- added REF**: MountingHole_4.3mm_M4_Pad, MountingHole:MountingHole_4.3mm_M4_Pad, F.Cu at (108.6, -19.0)
- added REF**: MountingHole_4.3mm_M4_Pad, MountingHole:MountingHole_4.3mm_M4_Pad, F.Cu at (107.0, -96.8)
- added REF**: MountingHole_4.3mm_M4_Pad, MountingHole:MountingHole_4.3mm_M4_Pad, F.Cu at (346.9, -16.2)
- added REF**: MountingHole_4.3mm_M4_Pad, MountingHole:MountingHole_4.3mm_M4_Pad, F.Cu at (347.2, -94.7)
- moved J28 289.1 mm to (318.5, -92.3), turned to 180 degrees
- moved U38 284.5 mm to (318.8, -73.9), turned to 180 degrees
- moved D11 283.8 mm to (278.8, -86.0), turned to 180 degrees
- moved J29 277.7 mm to (323.8, -16.2)
- moved J30 277.7 mm to (311.8, -16.2)
- moved U12 270.0 mm to (267.0, -76.4), turned to 90 degrees
- moved U11 269.8 mm to (279.0, -76.4), turned to 90 degrees
- moved U14 247.1 mm to (243.0, -76.4), turned to 90 degrees
- moved R18 244.0 mm to (279.0, -67.6), turned to 180 degrees
- moved D12 240.1 mm to (266.8, -86.0), turned to 180 degrees
- moved U9 234.6 mm to (265.4, -31.5), turned to -90 degrees
- moved U13 225.0 mm to (255.0, -76.4), turned to 90 degrees
- moved U15 224.0 mm to (231.0, -76.4), turned to 90 degrees
- moved D16 223.6 mm to (218.8, -86.0), turned to 180 degrees
- moved U8 221.1 mm to (253.4, -31.5), turned to -90 degrees
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
Commit message: Group components
Parts:
- added C50: 22uF, Capacitor_SMD:C_1206_3216Metric, F.Cu at (243.4, 160.2)
- U21, U22, U23, U24, U25, U26, U29, U30: value OPTO_TLP2366_V4-TPL,E -> TLP2366
- moved D49 348.4 mm to (326.0, -87.1)
- moved R90 333.2 mm to (325.4, -80.2), turned to -90 degrees
- moved D46 329.8 mm to (317.7, -72.8)
- moved D48 316.0 mm to (317.1, -84.9)
- moved Q2 315.6 mm to (326.4, -84.1), turned to 180 degrees
- moved R91 310.6 mm to (329.3, -87.1), turned to 180 degrees
- moved R92 280.7 mm to (329.5, -84.2), turned to 90 degrees
- moved R89 272.3 mm to (321.1, -85.0)
- moved R55 202.3 mm to (29.2, -53.1)
- moved C15 200.5 mm to (29.4, -44.8)
- moved U29 190.0 mm to (29.5, -49.2)
- moved U34 185.3 mm to (243.9, 104.9)
- moved R54 181.5 mm to (64.1, -53.9)
- moved C21 179.2 mm to (66.9, -55.2), turned to -90 degrees
- moved C29 172.6 mm to (247.3, 96.4)
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
Commit message: Modified de-safing key arrangement
Parts:
- added REF**: AMASS_XT60-M_1x02_P7.20mm_Vertical, Connector_AMASS:AMASS_XT60-M_1x02_P7.20mm_Vertical, F.Cu at (362.9, -40.6)
- added REF**: MountingHole_3.2mm_M3_Pad, MountingHole:MountingHole_3.2mm_M3_Pad, F.Cu at (95.4, -19.5)
- added REF**: AMASS_XT60PW-M_1x02_P7.20mm_Horizontal, Connector_AMASS:AMASS_XT60PW-M_1x02_P7.20mm_Horizontal, F.Cu at (360.7, -27.9)
- added REF**: MountingHole_3.2mm_M3_Pad, MountingHole:MountingHole_3.2mm_M3_Pad, F.Cu at (96.6, -97.5)
Changed lines of the file:
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@@
     )
   )
+  (footprint "Connector_AMASS:AMASS_XT60-M_1x02_P7.20mm_Vertical" (layer "F.Cu")
+    (at 362.9 -40.6)
+    (descr "AMASS female XT60, through hole, vertical, https://www.tme.eu/Document/2d152ced3b7a446066e6c419d84bb460/XT60%20SPEC.pdf")
+    (tags "XT60 female vertical")
+    (attr through_hole)
+    (fp_text reference "REF**" (at 3.6 -5.3 180) (layer "F.SilkS")
+      (effects (font (size 1 1) (thickness 0.15)))
+    )
+    (fp_text value "AMASS_XT60-M_1x02_P7.20mm_Vertical" (at 3.6 5.4) (layer "F.Fab")
+      (effects (font (size 1 1) (thickness 0.15)))
+    )
+    (fp_text user "${REFERENCE}" (at 3.6 0.05) (layer "F.Fab")
+      (effects (font (size 1 1) (thickness 0.15)))
+    )
+    (fp_line (start -4.25 1.55) (end -1.4 4.15) (layer "F.SilkS") (width 0.12))
+    (fp_line (start 11.45 4.15) (end 11.45 -4.15) (layer "F.SilkS") (width 0.12))
+    (fp_line (start -4.25 -1.6) (end -4.25 1.55) (layer "F.SilkS") (width 0.12))
+    (fp_line (start -1.4 -4.15) (end -4.25 -1.6) (layer "F.SilkS") (width 0.12))
+    (fp_line (start -1.4 4.15) (end 11.45 4.15) (layer "F.SilkS") (width 0.12))
+    (fp_line (start 11.45 -4.15) (end -1.4 -4.15) (layer "F.SilkS") (width 0.12))
+    (fp_line (start 11.85 4.6) (end -1.6 4.6) (layer "F.CrtYd") (width 0.05))
+    (fp_line (start -1.6 -4.6) (end 11.85 -4.6) (layer "F.CrtYd") (width 0.05))
+    (fp_line (start -4.65 1.85) (end -4.65 -1.85) (layer "F.CrtYd") (width 0.05))
+    (fp_line (start 11.85 -4.6) (end 11.85 4.6) (layer "F.CrtYd") (width 0.05))
+    (fp_line (start -1.6 4.6) (end -4.65 1.85) (layer "F.CrtYd") (width 0.05))
+    (fp_line (start -4.65 -1.85) (end -1.6 -4.6) (layer "F.CrtYd") (width 0.05))
+    (fp_line (start -4.15 -1.55) (end -4.15 1.55) (layer "F.Fab") (width 0.12))
+    (fp_line (start -4.15 1.55) (end -1.4 4.05) (layer "F.Fab") (width 0.12))
+    (fp_line (start 11.35 -4.05) (end -1.4 -4.05) (layer "F.Fab") (width 0.12))
+    (fp_line (start 11.35 4.05) (end 11.35 -4.05) (layer "F.Fab") (width 0.12))
+    (fp_line (start -1.4 4.05) (end 11.35 4.05) (layer "F.Fab") (width 0.12))
+    (fp_line (start -1.4 -4.05) (end -4.15 -1.55) (layer "F.Fab") (width 0.12))
+    (pad "1" thru_hole roundrect (at 0 0) (size 6 6) (drill 4.5) (layers *.Cu *.Mask) (roundrect_rratio 0.25))
+    (pad "2" thru_hole circle (at 7.2 0) (size 6 6) (drill 4.5) (layers *.Cu *.Mask))
+    (model "${KICAD6_3DMODEL_DIR}/Connector_AMASS.3dshapes/AMASS_XT60-M_1x02_P7.2mm_Vertical.wrl"
+      (offset (xyz 0 0 0))
+      (scale (xyz 1 1 1))
+      (rotate (xyz 0 0 0))
+    )
+  )
   (footprint "Resistor_SMD:R_0603_1608Metric" (layer "F.Cu")
     (at 131.6 46.4)
@@
     )
   )
+  (footprint "MountingHole:MountingHole_3.2mm_M3_Pad" (layer "F.Cu")
+    (at 95.4 -19.5)
+    (descr "Mounting Hole 3.2mm, M3")
+    (tags "mounting hole 3.2mm m3")
+    (attr exclude_from_pos_files exclude_from_bom)
+    (fp_text reference "REF**" (at 0 -4.2) (layer "F.SilkS")
+      (effects (font (size 1 1) (thickness 0.15)))
+    )
+    (fp_text value "MountingHole_3.2mm_M3_Pad" (at 0 4.2) (layer "F.Fab")
+      (effects (font (size 1 1) (thickness 0.15)))
+    )
+    (fp_text user "${REFERENCE}" (at 0 0) (layer "F.Fab")
+      (effects (font (size 1 1) (thickness 0.15)))
+    )
+    (fp_circle (center 0 0) (end 3.2 0) (layer "Cmts.User") (width 0.15) (fill none))
+    (fp_circle (center 0 0) (end 3.45 0) (layer "F.CrtYd") (width 0.05) (fill none))
+    (pad "1" thru_hole circle (at 0 0) (size 6.4 6.4) (drill 3.2) (layers *.Cu *.Mask))
+  )
   (footprint "Resistor_SMD:R_0603_1608Metric" (layer "F.Cu")
     (at 271.4 31.9)
@@
     )
   )
+  (footprint "Connector_AMASS:AMASS_XT60PW-M_1x02_P7.20mm_Horizontal" (layer "F.Cu")
+    (at 360.7 -27.9 -90)
+    (descr "Connector XT60 Horizontal PCB Female, https://www.tme.eu/en/Document/9b8d0c5eb7094295f3d3112c214d3ade/XT60PW%20SPEC.pdf")
+    (tags "RC Connector XT60")
+    (attr through_hole)
+    (fp_text reference "REF**" (at 3.6 -17.5 90) (layer "F.SilkS")
+      (effects (font (size 1 1) (thickness 0.15)))
+    )
+    (fp_text value "AMASS_XT60PW-M_1x02_P7.20mm_Horizontal" (at 3.6 4 90) (layer "F.Fab")
+      (effects (font (size 1 1) (thickness 0.15)))
+    )
+    (fp_text user "+" (at 9.5 2.5 90) (layer "F.SilkS")
+      (effects (font (size 1.5 1.5) (thickness 0.15)))
+    )
+    (fp_text user "-" (at -2.8 2.5 90) (layer "F.SilkS")
+      (effects (font (size 1.5 1.5) (thickness 0.15)))
+    )
+    (fp_text user "${REFERENCE}" (at 3.6 -3.6 90) (layer "F.Fab")
+      (effects (font (size 1 1) (thickness 0.15)))
+    )
+    (fp_line (start 2.31 1.96) (end 6.05 1.96) (layer "F.SilkS") (width 0.12))
+    (fp_line (start 11.46 -16.46) (end 11.46 -2.15) (layer "F.SilkS") (width 0.12))
+    (fp_line (start -4.26 -16.46) (end -4.26 -2.15) (layer "F.SilkS") (width 0.12))
+    (fp_line (start -4.26 -16.46) (end 11.46 -16.46) (layer "F.SilkS") (width 0.12))
+    (fp_arc (start -2.266806 1.372958) (mid -3.727162 -0.126139) (end -4.26 -2.15) (layer "F.SilkS") (width 0.12))
+    (fp_arc (start 11.46 -2.15) (mid 10.653852 0.294722) (end 8.551648 1.780413) (layer "F.SilkS") (width 0.12))
+    (fp_line (start -4.65 -16.85) (end -4.65 2.55) (layer "F.CrtYd") (width 0.05))
+    (fp_line (start -4.65 -16.85) (end 11.85 -16.85) (layer "F.CrtYd") (width 0.05))
+    (fp_line (start 11.85 -16.85) (end 11.85 2.55) (layer "F.CrtYd") (width 0.05))
+    (fp_line (start 11.85 2.55) (end -4.65 2.55) (layer "F.CrtYd") (width 0.05))
+    (fp_line (start -4.15 -16.35) (end -4.15 -2.15) (layer "F.Fab") (width 0.1))
+    (fp_line (start -0.15 1.85) (end 7.35 1.85) (layer "F.Fab") (width 0.1))
+    (fp_line (start 11.35 -16.35) (end 11.35 -2.15) (layer "F.Fab") (width 0.1))
+    (fp_line (start -4.15 -16.35) (end 11.35 -16.35) (layer "F.Fab") (width 0.1))
+    (fp_arc (start 11.35 -2.15) (mid 10.178427 0.678427) (end 7.35 1.85) (layer "F.Fab") (width 0.1))
+    (fp_arc (start -0.15 1.85) (mid -2.978427 0.678427) (end -4.15 -2.15) (layer "F.Fab") (width 0.1))
+    (pad "" thru_hole rect (at -3.15 -6 270) (size 0.9 2) (drill oval 0.6 1.7) (layers *.Cu *.Mask))
+    (pad "" thru_hole rect (at 10.35 -6 270) (size 0.9 2) (drill oval 0.6 1.7) (layers *.Cu *.Mask))
+    (pad "1" thru_hole roundrect (at 0 0 270) (size 4.1 4.1) (drill 2.7) (layers *.Cu *.Mask) (roundrect_rratio 0.25))
+    (pad "2" thru_hole circle (at 7.2 0 270) (size 4.1 4.1) (drill 2.7) (layers *.Cu *.Mask))
+    (model "${KICAD6_3DMODEL_DIR}/Connector_AMASS.3dshapes/AMASS_XT60PW-M_1x02_P7.20mm_Horizontal.wrl"
+      (offset (xyz 0 0 0))
+      (scale (xyz 1 1 1))
+      (rotate (xyz 0 0 0))
+    )
+  )
   (footprint "LED_SMD:LED_0603_1608Metric" (layer "F.Cu")
     (at 138.4 41.3)
@@
     )
   )
+  (footprint "MountingHole:MountingHole_3.2mm_M3_Pad" (layer "F.Cu")
+    (at 96.6 -97.5)
+    (descr "Mounting Hole 3.2mm, M3")
+    (tags "mounting hole 3.2mm m3")
+    (attr exclude_from_pos_files exclude_from_bom)
+    (fp_text reference "REF**" (at 0 -4.2) (layer "F.SilkS")
+      (effects (font (size 1 1) (thickness 0.15)))
+    )
+    (fp_text value "MountingHole_3.2mm_M3_Pad" (at 0 4.2) (layer "F.Fab")
+      (effects (font (size 1 1) (thickness 0.15)))
+    )
+    (fp_text user "${REFERENCE}" (at 0 0) (layer "F.Fab")
+      (effects (font (size 1 1) (thickness 0.15)))
+    )
+    (fp_circle (center 0 0) (end 3.2 0) (layer "Cmts.User") (width 0.15) (fill none))
+    (fp_circle (center 0 0) (end 3.45 0) (layer "F.CrtYd") (width 0.05) (fill none))
+    (pad "1" thru_hole circle (at 0 0) (size 6.4 6.4) (drill 3.2) (layers *.Cu *.Mask))
+  )
   (footprint "Resistor_SMD:R_0603_1608Metric" (layer "F.Cu")

Commit message: Check-safe channel, footprint changes
Parts:
- removed the REF** at (362.9, -40.6)
- removed the REF** at (360.7, -27.9)
- added REF**: CP_Elec_6.3x5.9, Capacitor_SMD:CP_Elec_6.3x5.9, F.Cu at (190.0, -107.7)
- added REF**: CP_Elec_4x5.8, Capacitor_SMD:CP_Elec_4x5.8, F.Cu at (188.2, -87.9)
- added REF**: CP_Elec_4x5.8, Capacitor_SMD:CP_Elec_4x5.8, F.Cu at (198.2, -87.9)
- J10, J11, J12, J13, J14, J15, J16, J17, J2, J3, J4, J5, J6, J7, J8, J9: footprint actuation:1989447 -> Connector_AMASS:AMASS_XT30U-M_1x02_P5.0mm_Vertical
- J24: footprint actuation:1773976 -> actuation:XT90PW-M
- J27: value SAFING -> SAFETY; footprint actuation:1773976 -> actuation:XT90PW-M
- J29, J30: footprint actuation:1989447 -> Connector_AMASS:AMASS_XT60-M_1x02_P7.20mm_Vertical
- moved R55 168.4 mm to (161.4, -157.4)
- moved R56 168.4 mm to (205.8, -154.9)
- moved C15 168.4 mm to (161.6, -149.1)
- moved C16 168.4 mm to (196.2, -149.8)
- moved C21 168.4 mm to (199.1, -159.5)
- moved C24 168.4 mm to (205.6, -150.1)
- moved R54 168.4 mm to (196.3, -158.2)
- moved R57 168.4 mm to (205.4, -152.3)
- moved U29 168.4 mm to (161.7, -153.5)
- moved U30 168.4 mm to (196.6, -153.7)
- moved U31 168.4 mm to (202.4, -159.5)
- moved C34 160.4 mm to (172.8, 94.7)
- moved C35 160.4 mm to (172.8, 97.6)
- moved R74 160.4 mm to (164.8, 111.8)
- moved C31 160.4 mm to (177.1, 110.9)
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Connections:
- J27 pad 1: Net-(J27-Pad1) -> VDC
- J27 pad 2: Vdrive -> Net-(J27-Pad2)
- K1 pad 1: VDC -> Net-(J27-Pad2)
- K1 pad 4: Net-(J27-Pad1) -> Vdrive

Commit message: placed power parts
Parts:
- removed J30: ACT COLD, Connector_AMASS:AMASS_XT60-M_1x02_P7.20mm_Vertical
- removed REF** (x4): MountingHole_4.3mm_M4_Pad, MountingHole:MountingHole_4.3mm_M4_Pad
- removed REF** (x2): MountingHole_3.2mm_M3_Pad, MountingHole:MountingHole_3.2mm_M3_Pad
- removed REF**: CP_Elec_6.3x5.9, Capacitor_SMD:CP_Elec_6.3x5.9
- removed REF** (x2): CP_Elec_4x5.8, Capacitor_SMD:CP_Elec_4x5.8
- added C51: 6.8nF, Capacitor_SMD:C_0603_1608Metric, F.Cu at (279.9, -307.5)
- added C52: 10uF, Capacitor_SMD:C_1206_3216Metric, F.Cu at (150.0, -244.3)
- added C53: 10uF, Capacitor_SMD:C_1206_3216Metric, F.Cu at (144.3, -244.3)
- added C54: 10nF, Capacitor_SMD:C_0603_1608Metric, F.Cu at (278.4, -314.9)
- added C55: 10nF, Capacitor_SMD:C_0603_1608Metric, F.Cu at (278.0, -307.6)
- added C56: 10uF, Capacitor_SMD:C_1206_3216Metric, F.Cu at (144.3, -237.6)
- added C57: 1uF, Capacitor_SMD:C_0603_1608Metric, F.Cu at (274.5, -307.6)
- added C58: 0.1uF, Capacitor_SMD:C_0603_1608Metric, F.Cu at (276.2, -307.6)
- added C59: 0.1uF, Capacitor_SMD:C_0603_1608Metric, F.Cu at (147.6, -230.3)
- added C60: 3.3nF, Capacitor_SMD:C_0603_1608Metric, F.Cu at (159.7, -230.6)
- added C61: 68nF, Capacitor_SMD:C_0603_1608Metric, F.Cu at (171.4, -245.2)
- added C62: 22uF, Capacitor_SMD:C_1206_3216Metric, F.Cu at (152.4, -248.9)
- added C63: 22uF, Capacitor_SMD:C_1206_3216Metric, F.Cu at (144.3, -241.0)
- added C64: 10uF, Capacitor_SMD:C_0805_2012Metric, F.Cu at (155.0, -245.7)
- added C65: 1uF, Capacitor_SMD:C_0603_1608Metric, F.Cu at (163.7, -232.1)
- added C66: 1uF, Capacitor_SMD:C_0603_1608Metric, F.Cu at (167.8, -237.1)
- added C67: 10uF, Capacitor_SMD:C_0805_2012Metric, F.Cu at (149.4, -241.1)
- added C68: 22uF, Capacitor_SMD:C_1206_3216Metric, F.Cu at (158.0, -248.9)
- added D52: SMAJ28CAQ-13-F, Diode_SMD:D_SMA, F.Cu at (293.1, -275.9)
- added R95: 470R, Resistor_SMD:R_0603_1608Metric, F.Cu at (254.4, -301.7)
- added R96: 10k, Resistor_SMD:R_0603_1608Metric, F.Cu at (252.3, -312.1)
- added R97: 10k, Resistor_SMD:R_0603_1608Metric, F.Cu at (271.2, -260.6)
- added R98: 470R, Resistor_SMD:R_0603_1608Metric, F.Cu at (171.4, -242.7)
- added TP1: TestPoint_Alt, TestPoint:TestPoint_Pad_D2.0mm, F.Cu at (215.0, -296.8)
- added TP10: TestPoint_Alt, TestPoint:TestPoint_Pad_D2.0mm, F.Cu at (299.1, -260.7)
- added TP11: TestPoint_Alt, TestPoint:TestPoint_Pad_D2.0mm, F.Cu at (294.2, -253.1)
- added TP12: TestPoint_Alt, TestPoint:TestPoint_Pad_D2.0mm, F.Cu at (314.7, -303.7)
- added TP13: TestPoint_Alt, TestPoint:TestPoint_Pad_D2.0mm, F.Cu at (143.5, -229.9)
- added TP14: TestPoint_Alt, TestPoint:TestPoint_Pad_D2.0mm, F.Cu at (314.7, -310.3)
- added TP15: TestPoint_Alt, TestPoint:TestPoint_Pad_D2.0mm, F.Cu at (314.8, -307.0)
- added TP16: TestPoint_Alt, TestPoint:TestPoint_Pad_D2.0mm, F.Cu at (155.7, -233.5)
- added TP17: TestPoint_Alt, TestPoint:TestPoint_Pad_D2.0mm, F.Cu at (149.2, -237.6)
- added TP18: TestPoint_Alt, TestPoint:TestPoint_Pad_D2.0mm, F.Cu at (314.7, -318.3)
- added TP19: TestPoint_Alt, TestPoint:TestPoint_Pad_D2.0mm, F.Cu at (159.7, -236.4)
- added TP2: TestPoint_Alt, TestPoint:TestPoint_Pad_D2.0mm, F.Cu at (143.5, -222.7)
- added TP20: TestPoint_Alt, TestPoint:TestPoint_Pad_D2.0mm, F.Cu at (298.7, -273.5)
- added TP21: TestPoint_Alt, TestPoint:TestPoint_Pad_D2.0mm, F.Cu at (314.6, -300.5)
- added TP22: TestPoint_Alt, TestPoint:TestPoint_Pad_D2.0mm, F.Cu at (143.5, -233.9)
- added TP23: TestPoint_Alt, TestPoint:TestPoint_Pad_D2.0mm, F.Cu at (281.4, -277.5)
- added TP24: TestPoint_Alt, TestPoint:TestPoint_Pad_D2.0mm, F.Cu at (251.4, -316.6)
- added TP25: TestPoint_Alt, TestPoint:TestPoint_Pad_D2.0mm, F.Cu at (158.9, -240.4)
- added TP26: TestPoint_Alt, TestPoint:TestPoint_Pad_D2.0mm, F.Cu at (247.1, -309.5)
- added TP27: TestPoint_Alt, TestPoint:TestPoint_Pad_D2.0mm, F.Cu at (171.0, -248.5)
- added TP3: TestPoint_Alt, TestPoint:TestPoint_Pad_D2.0mm, F.Cu at (147.6, -222.7)
- added TP4: TestPoint_Alt, TestPoint:TestPoint_Pad_D2.0mm, F.Cu at (195.2, -248.5)
- added TP5: TestPoint_Alt, TestPoint:TestPoint_Pad_D2.0mm, F.Cu at (187.1, -244.5)
- added TP6: TestPoint_Alt, TestPoint:TestPoint_Pad_D2.0mm, F.Cu at (191.1, -244.5)
- added TP7: TestPoint_Alt, TestPoint:TestPoint_Pad_D2.0mm, F.Cu at (191.1, -248.5)
- added TP8: TestPoint_Alt, TestPoint:TestPoint_Pad_D2.0mm, F.Cu at (187.1, -248.5)
- added TP9: TestPoint_Alt, TestPoint:TestPoint_Pad_D2.0mm, F.Cu at (284.1, -314.5)
- added U40: LP5912-3.3DRV, Package_SON:WSON-6-1EP_2x2mm_P0.65mm_EP1x1.6mm, F.Cu at (167.6, -234.1)
- C10, C11, C12, C13, C14, C15, C16, C19, C20, C7, C8, C9: value 0.1uF -> 10uF; footprint Capacitor_SMD:C_0603_1608Metric -> Capacitor_SMD:CP_Elec_4x5.8
- C17, C18: value 1nF -> 10uF; footprint Capacitor_SMD:C_0603_1608Metric -> Capacitor_SMD:CP_Elec_4x5.8
- C21, C22: value 0.1uF -> 1uF
- C25, C26, C29, C39, C48: value 1uF -> 0.1uF
- C31: value 6nF -> 0.1uF
- C32: value 6.8nF -> 0.1uF
- C33: value 6.8nF -> 1nF
- C34: value 10uF -> 1nF; footprint Capacitor_SMD:C_1206_3216Metric -> Capacitor_SMD:C_0603_1608Metric
- C35, C38: value 10uF -> 0.1uF; footprint Capacitor_SMD:C_1206_3216Metric -> Capacitor_SMD:C_0603_1608Metric
- C36, C37: value 10nF -> 0.1uF
- C42: value 3.3nF -> 0.1uF
- C43: value 68nF -> 1uF
- C44: value 22uF -> 1uF; footprint Capacitor_SMD:C_1206_3216Metric -> Capacitor_SMD:C_0603_1608Metric
- C45: value 22uF -> 0.1uF; footprint Capacitor_SMD:C_1206_3216Metric -> Capacitor_SMD:C_0603_1608Metric
- C46: value 10uF -> 0.1uF; footprint Capacitor_SMD:C_0805_2012Metric -> Capacitor_SMD:C_0603_1608Metric
- C49: value 10uF -> 6nF; footprint Capacitor_SMD:C_0805_2012Metric -> Capacitor_SMD:C_0603_1608Metric
- C5, C6: value 1uF -> 10uF; footprint Capacitor_SMD:C_0603_1608Metric -> Capacitor_SMD:CP_Elec_4x5.8
- C50: value 22uF -> 6.8nF; footprint Capacitor_SMD:C_1206_3216Metric -> Capacitor_SMD:C_0603_1608Metric
- D37: value FB CH1 -> CHK SAF
- D38: value FB CH2 -> FB CH1
- D39: value FB CH3 -> FB CH2
- D40: value FB CH4 -> FB CH3
- J21: value FB CH4 -> VDET CH1; footprint actuation:1751251 -> actuation:1751248
- J22: value VDET CH1 -> VDET CH2
- J23: value VDET CH2 -> PWR IN; footprint actuation:1751248 -> actuation:XT90PW-M
- J24: value PWR IN -> PWR PROT; footprint actuation:XT90PW-M -> Connector_AMASS:AMASS_XT60-M_1x02_P7.20mm_Vertical
- J25: value PWR PROT -> PWR 3.3V; footprint actuation:1989447 -> Connector_AMASS:AMASS_XT60-M_1x02_P7.20mm_Vertical
- J26: value PWR 3.3V -> SAFETY; footprint actuation:1989447 -> actuation:XT90PW-M
- J27: value SAFETY -> ARM; footprint actuation:XT90PW-M -> Connector_AMASS:AMASS_XT60-M_1x02_P7.20mm_Vertical
- J28: value ARM -> ACT HOT; footprint actuation:1989447 -> Connector_AMASS:AMASS_XT60-M_1x02_P7.20mm_Vertical
- J29: value ACT HOT -> ACT COLD
- R58: value 470R -> 100k
- R59: value 470R -> 13k
- R66, R67: value 4.7k -> 470R
- R74: value 1.87M -> 4.7k
- R75: value 32.4k -> 4.7k
- R76: value 510k -> 1.87M
- R77: value 10R -> 32.4k
- R78: value 10R -> 510k
- R79: value 5.1k -> 10R
- R80: value 270R -> 10R
- R81: value 270R -> 5.1k
- R82, R94: value 470R -> 270R
- R83: value 200k -> 270R
- R84: value 10k -> 470R
- R85: value 9.31k -> 200k
- R86: value 69.8k -> 10k
- R87: value 22.1k -> 9.31k
- R88: value 1k -> 69.8k
- R89: value 4.7k -> 22.1k
- R90: value 270R -> 47k
- R91: value 470R -> 47k
- R92: value 10k -> 1k
- R93: value 10k -> 4.7k
- U32: value PCA9534 -> 74LVC1G126; footprint Package_SO:TSSOP-16_4.4x5mm_P0.65mm -> Package_TO_SOT_SMD:SOT-23-5
- U33: value SN74LVC541A -> PCA9534; footprint Package_SO:TSSOP-20_4.4x6.5mm_P0.65mm -> Package_SO:TSSOP-16_4.4x5mm_P0.65mm
- U34: value TLI4971 -> SN74LVC541A; footprint Package_SON:Infineon_PG-TISON-8-5 -> Package_SO:TSSOP-20_4.4x6.5mm_P0.65mm
- U35: value LTC4367 -> TLI4971; footprint Package_DFN_QFN:DFN-8-1EP_3x3mm_P0.5mm_EP1.65x2.38mm -> Package_SON:Infineon_PG-TISON-8-5
- U36: value ADS1110 -> LTC4367; footprint Package_TO_SOT_SMD:SOT-23-6 -> Package_DFN_QFN:DFN-8-1EP_3x3mm_P0.5mm_EP1.65x2.38mm
- U37: value AP64350 -> ADS1110; footprint Package_SO:SOIC-8-1EP_3.9x4.9mm_P1.27mm_EP2.62x3.51mm -> Package_TO_SOT_SMD:SOT-23-6
- U38: value TLP241A -> AP64350; footprint actuation:TLP241A -> Package_SO:SOIC-8-1EP_3.9x4.9mm_P1.27mm_EP2.62x3.51mm
- U39: value LP5912-3.3DRV -> TLP241A; footprint Package_SON:WSON-6-1EP_2x2mm_P0.65mm_EP1x1.6mm -> actuation:TLP241A
- moved R86 549.1 mm to (312.1, -314.1)
- moved R83 533.0 mm to (279.0, -310.4), turned to 180 degrees
- moved U37 523.7 mm to (275.6, -311.5), turned to -90 degrees
- moved R82 523.7 mm to (279.0, -312.1), turned to 180 degrees
- moved R4 513.5 mm to (210.1, -314.1), turned to -90 degrees
- moved D2 511.4 mm to (240.9, -327.8), turned to -90 degrees
- moved D1 509.6 mm to (243.3, -327.8), turned to -90 degrees
- moved R3 509.5 mm to (213.8, -313.4), turned to -90 degrees
- moved R7 508.3 mm to (209.9, -309.4), turned to -90 degrees
- moved R2 504.8 mm to (218.4, -312.6), turned to -90 degrees
- moved R6 504.1 mm to (214.3, -309.0), turned to -90 degrees
- moved R1 500.8 mm to (225.9, -314.4), turned to -90 degrees
- moved U1 500.2 mm to (215.2, -306.1), turned to 90 degrees
- moved R5 500.1 mm to (218.6, -308.6), turned to -90 degrees
- moved U2 496.1 mm to (209.9, -303.1), turned to 90 degrees
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Connections:
- C10 pad 1: +3.3V -> Vdrive
- C10 pad 2: GND -> GNDPWR
- C11 pad 1: +3.3V -> Vdrive
- C11 pad 2: GND -> GNDPWR
- C12 pad 1: +3.3V -> Vdrive
- C12 pad 2: GND -> GNDPWR
- C13 pad 1: +3.3V -> Vdrive
- C13 pad 2: GND -> GNDPWR
- C14 pad 1: +3.3V -> Vdrive
- C14 pad 2: GND -> GNDPWR
- C15 pad 1: +3.3V -> Vdrive
- C15 pad 2: GND -> GNDPWR
- C16 pad 1: +3.3V -> Vdrive
- C16 pad 2: GND -> GNDPWR
- C17 pad 1: Net-(C17-Pad1) -> Vdrive
- C17 pad 2: Net-(C17-Pad2) -> GNDPWR
- C18 pad 1: Net-(C18-Pad1) -> Vdrive
- C18 pad 2: Net-(C18-Pad2) -> GNDPWR
- C19 pad 1: Net-(C17-Pad1) -> Vdrive
- C20 pad 1: Net-(C18-Pad1) -> Vdrive
- C21 pad 1: 3.3V_ACT -> +3.3V
- C21 pad 2: GNDPWR -> GND
- C22 pad 1: 3.3V_ACT -> +3.3V
- C22 pad 2: GNDPWR -> GND
- C23 pad 1: 3.3V_ACT -> +3.3V
- C23 pad 2: GNDPWR -> GND
- C24 pad 1: Net-(C24-Pad1) -> +3.3V
- C24 pad 2: GNDPWR -> GND
- C31 pad 1: Net-(C31-Pad1) -> +3.3V
- C31 pad 2: GNDPWR -> GND
- C32 pad 1: Net-(C32-Pad1) -> +3.3V
- C33 pad 2: GND -> Net-(C33-Pad2)
- C34 pad 1: VBUS -> Net-(C34-Pad1)
- C34 pad 2: GNDPWR -> Net-(C34-Pad2)
- C35 pad 1: VBUS -> Net-(C33-Pad1)
- C36 pad 1: Net-(C36-Pad1) -> Net-(C34-Pad1)
- C36 pad 2: GND -> GNDPWR
- C37 pad 1: Net-(C37-Pad1) -> 3.3V_ACT
- C37 pad 2: GND -> GNDPWR
- C38 pad 1: VBUS -> 3.3V_ACT
- C39 pad 1: +3.3V -> 3.3V_ACT
- C39 pad 2: GND -> GNDPWR
- C40 pad 1: +3.3V -> 3.3V_ACT
- C40 pad 2: GND -> GNDPWR
- C41 pad 2: Net-(C41-Pad2) -> GNDPWR
- C43 pad 1: Net-(C43-Pad1) -> +3.3V
- C43 pad 2: GNDPWR -> GND
- C44 pad 1: 3.3V_ACT -> +3.3V
- C44 pad 2: GNDPWR -> GND
- C45 pad 1: 3.3V_ACT -> +3.3V
- C45 pad 2: GNDPWR -> GND
- C46 pad 1: +5V -> +3.3V
- C47 pad 1: +5V -> +3.3V
- C49 pad 1: +3.3V -> Net-(C49-Pad1)
- C49 pad 2: GND -> GNDPWR
- C5 pad 1: +3.3V -> Vdrive
- C5 pad 2: GND -> GNDPWR
- C50 pad 1: GND -> Net-(C50-Pad1)
- C50 pad 2: +3.3V -> GND
- C6 pad 1: +3.3V -> Vdrive
- C6 pad 2: GND -> GNDPWR
- C7 pad 1: +3.3V -> Vdrive
- C7 pad 2: GND -> GNDPWR
- C8 pad 1: +3.3V -> Vdrive
- C8 pad 2: GND -> GNDPWR
- C9 pad 1: +3.3V -> Vdrive
- C9 pad 2: GND -> GNDPWR
- J21 pad 1: 3.3V_ACT -> Net-(J21-Pad1)
- J21 pad 2: Net-(J21-Pad2) -> GNDPWR
- J24 pad 1: Net-(J24-Pad1) -> VBUS
- J25 pad 1: VBUS -> 3.3V_ACT
- J26 pad 1: 3.3V_ACT -> VDC
- J26 pad 2: GNDPWR -> VDESAFED
- J27 pad 1: VDC -> Net-(J27-Pad1)
- J27 pad 2: Net-(J27-Pad2) -> Net-(D46-Pad2)
- J28 pad 1: Net-(J28-Pad1) -> Vdrive
- J28 pad 2: Net-(D46-Pad2) -> GNDPWR
- J29 pad 1: Vdrive -> VCOLD
- K1 pad 1: Net-(J27-Pad2) -> VDESAFED
- K1 pad 5: VSAFE -> VCOLD
- L1 pad 1: Net-(C41-Pad2) -> Net-(C59-Pad2)
- R44 pad 2: Net-(J18-Pad2) -> 3.3V_ACT
- R45 pad 2: Net-(J19-Pad2) -> Net-(J18-Pad2)
- R46 pad 2: Net-(J20-Pad2) -> Net-(J19-Pad2)
- R47 pad 2: Net-(J21-Pad2) -> Net-(J20-Pad2)
- R48 pad 2: Net-(C17-Pad2) -> Net-(C33-Pad2)
- R49 pad 1: Net-(C17-Pad2) -> Net-(C33-Pad2)
- R50 pad 2: Net-(C18-Pad2) -> Net-(C34-Pad2)
- R51 pad 1: Net-(C18-Pad2) -> Net-(C34-Pad2)
- R52 pad 1: Net-(C17-Pad1) -> Net-(C33-Pad1)
- R52 pad 2: Net-(J22-Pad1) -> Net-(J21-Pad1)
- R53 pad 1: Net-(C18-Pad1) -> Net-(C34-Pad1)
- R53 pad 2: Net-(J23-Pad1) -> Net-(J22-Pad1)
- R55 pad 2: 3.3V_ACT -> Net-(R55-Pad2)
- R56 pad 2: Net-(C24-Pad1) -> Net-(C41-Pad1)
- R57 pad 1: Net-(C24-Pad1) -> Net-(C41-Pad1)
- R58 pad 1: /Feedback Channels/FB_CH1_LED -> VDESAFED
- R58 pad 2: Net-(D35-Pad2) -> Net-(C42-Pad1)
- R59 pad 1: /Feedback Channels/FB_CH2_LED -> Net-(C42-Pad1)
- R59 pad 2: Net-(D36-Pad2) -> GNDPWR
- R60 pad 1: /Feedback Channels/FB_CH3_LED -> /Feedback Channels/FB_CH1_LED
- R60 pad 2: Net-(D37-Pad2) -> Net-(D35-Pad2)
- R61 pad 1: /Feedback Channels/FB_CH4_LED -> /Feedback Channels/FB_CH2_LED
- R61 pad 2: Net-(D38-Pad2) -> Net-(D36-Pad2)
- R62 pad 1: /Feedback Channels/FB_CH5_LED -> /Feedback Channels/FB_CH3_LED
- R62 pad 2: Net-(D39-Pad2) -> Net-(D37-Pad2)
- R63 pad 1: /Feedback Channels/FB_CH6_LED -> /Feedback Channels/FB_CH4_LED
- R63 pad 2: Net-(D40-Pad2) -> Net-(D38-Pad2)
- R64 pad 1: /Feedback Channels/FB_CH7_LED -> /Feedback Channels/FB_CH5_LED
- R64 pad 2: Net-(D41-Pad2) -> Net-(D39-Pad2)
- R65 pad 1: /Feedback Channels/FB_CH8_LED -> /Feedback Channels/FB_CH6_LED
- R65 pad 2: Net-(D42-Pad2) -> Net-(D40-Pad2)
- R66 pad 1: Net-(R66-Pad1) -> /Feedback Channels/FB_CH7_LED
- R66 pad 2: /Feedback Channels/FB_CH1 -> Net-(D41-Pad2)
- R67 pad 1: Net-(R67-Pad1) -> /Feedback Channels/FB_CH8_LED
- R67 pad 2: /Feedback Channels/FB_CH2 -> Net-(D42-Pad2)
- R68 pad 2: /Feedback Channels/FB_CH3 -> /Feedback Channels/FB_CH1
- R69 pad 2: /Feedback Channels/FB_CH4 -> /Feedback Channels/FB_CH2
- R70 pad 2: /Feedback Channels/FB_CH5 -> /Feedback Channels/FB_CH3
- R71 pad 2: /Feedback Channels/FB_CH6 -> /Feedback Channels/FB_CH4
- R72 pad 2: /Feedback Channels/FB_CH7 -> /Feedback Channels/FB_CH5
- R73 pad 2: /Feedback Channels/FB_CH8 -> /Feedback Channels/FB_CH6
- R74 pad 2: VDC -> /Feedback Channels/FB_CH7
- R75 pad 1: GNDPWR -> Net-(R75-Pad1)
- R75 pad 2: Net-(R74-Pad1) -> /Feedback Channels/FB_CH8
- R77 pad 1: Net-(Q1-Pad2) -> GNDPWR
- R77 pad 2: Net-(R77-Pad2) -> Net-(R76-Pad1)
- R78 pad 1: Net-(Q1-Pad4) -> Net-(R78-Pad1)
- R78 pad 2: Net-(R77-Pad2) -> VDC
- R79 pad 1: Net-(R77-Pad2) -> Net-(Q1-Pad2)
- R79 pad 2: Net-(C31-Pad1) -> Net-(R79-Pad2)
- R80 pad 1: Net-(C32-Pad1) -> Net-(Q1-Pad4)
- R80 pad 2: Net-(C36-Pad1) -> Net-(R79-Pad2)
- R81 pad 1: Net-(C33-Pad1) -> Net-(R79-Pad2)
- R81 pad 2: Net-(C37-Pad1) -> Net-(C49-Pad1)
- R82 pad 1: 3.3V_ACT -> Net-(C50-Pad1)
- R82 pad 2: Net-(D44-Pad2) -> Net-(C54-Pad1)
- R83 pad 1: Net-(R83-Pad1) -> Net-(C51-Pad1)
- R83 pad 2: GNDPWR -> Net-(C55-Pad1)
- R84 pad 1: VDC -> 3.3V_ACT
- R84 pad 2: Net-(D45-Pad2) -> Net-(D44-Pad2)
- R85 pad 1: Net-(C43-Pad1) -> Net-(R85-Pad1)
- R85 pad 2: Net-(C42-Pad1) -> GNDPWR
- R86 pad 1: 3.3V_ACT -> VDC
- R86 pad 2: Net-(R86-Pad2) -> Net-(D45-Pad2)
- R87 pad 1: Net-(R86-Pad2) -> Net-(C61-Pad1)
- R87 pad 2: GNDPWR -> Net-(C60-Pad1)
- R88 pad 1: +5V -> 3.3V_ACT
- R88 pad 2: Net-(D47-Pad2) -> Net-(R88-Pad2)
- R89 pad 1: Net-(J28-Pad1) -> Net-(R88-Pad2)
- R89 pad 2: Net-(D48-Pad2) -> GNDPWR
- R90 pad 1: +3.3V -> VDESAFED
- R90 pad 2: Net-(R90-Pad2) -> GNDPWR
- R91 pad 1: +3.3V -> Vdrive
- R91 pad 2: Net-(D49-Pad2) -> GNDPWR
- R92 pad 1: /ENERGIZE -> +5V
- R92 pad 2: GND -> Net-(D47-Pad2)
- R93 pad 1: Vdrive -> Net-(J27-Pad1)
- R93 pad 2: Net-(D50-Pad2) -> Net-(D48-Pad2)
- R94 pad 2: Net-(D51-Pad2) -> Net-(R94-Pad2)
- RV1 pad 3: Net-(C17-Pad1) -> Net-(C33-Pad1)
- RV2 pad 3: Net-(C18-Pad1) -> Net-(C34-Pad1)
- U19 pad 13: unconnected-(U19-Pad13) -> Net-(TP3-Pad1)
- U2 pad 3: unconnected-(U2-Pad3) -> Net-(TP1-Pad1)
- U20 pad 13: unconnected-(U20-Pad13) -> Net-(TP2-Pad1)
- U21 pad 5: /Feedback Channels/FB_CH3 -> /Feedback Channels/FB_CH1
- U27 pad 3: Net-(C17-Pad1) -> Net-(C33-Pad1)
- U27 pad 4: Net-(C17-Pad2) -> Net-(C33-Pad2)
- U28 pad 3: Net-(C18-Pad1) -> Net-(C34-Pad1)
- U28 pad 4: Net-(C18-Pad2) -> Net-(C34-Pad2)
- U29 pad 1: Net-(R55-Pad1) -> Net-(R54-Pad2)
- U29 pad 5: /Feedback Channels/FB_CH1 -> /Feedback Channels/FB_CH2
- U30 pad 1: Net-(R54-Pad2) -> Net-(R55-Pad2)
- U30 pad 5: /Feedback Channels/FB_CH2 -> /Feedback Channels/FB_CH3
- U31 pad 2: Net-(C24-Pad1) -> Net-(C41-Pad1)
- U32 pad 1: GND -> 3.3V_ACT
- U32 pad 2: +3.3V -> Net-(C42-Pad1)
- U32 pad 3: GND -> GNDPWR
- U32 pad 4: Net-(R66-Pad1) -> Net-(R55-Pad1)
- U32 pad 5: Net-(R67-Pad1) -> 3.3V_ACT
- U33 pad 10: GND -> Net-(R73-Pad1)
- U33 pad 11: /Feedback Channels/FB_CH8_LED -> Net-(R74-Pad1)
- U33 pad 12: /Feedback Channels/FB_CH7_LED -> Net-(R75-Pad1)
- U33 pad 13: /Feedback Channels/FB_CH6_LED -> Net-(TP8-Pad1)
- U33 pad 14: /Feedback Channels/FB_CH5_LED -> /SCL
- U33 pad 15: /Feedback Channels/FB_CH4_LED -> /SDA
- U33 pad 16: /Feedback Channels/FB_CH3_LED -> +3.3V
- U33 pad 2: /Feedback Channels/FB_CH1 -> +3.3V
- U33 pad 3: /Feedback Channels/FB_CH2 -> GND
- U33 pad 4: /Feedback Channels/FB_CH3 -> Net-(R68-Pad1)
- U33 pad 5: /Feedback Channels/FB_CH4 -> Net-(R69-Pad1)
- U33 pad 6: /Feedback Channels/FB_CH5 -> Net-(R70-Pad1)
- U33 pad 7: /Feedback Channels/FB_CH6 -> Net-(R71-Pad1)
- U33 pad 8: /Feedback Channels/FB_CH7 -> GND
- U33 pad 9: /Feedback Channels/FB_CH8 -> Net-(R72-Pad1)
- U34 pad 1: +3.3V -> GND
- U34 pad 2: GND -> /Feedback Channels/FB_CH1
- U34 pad 3: Net-(C33-Pad1) -> /Feedback Channels/FB_CH2
- U34 pad 4: Net-(C32-Pad1) -> /Feedback Channels/FB_CH3
- U34 pad 5: unconnected-(U34-Pad5) -> /Feedback Channels/FB_CH4
- U34 pad 6: unconnected-(U34-Pad6) -> /Feedback Channels/FB_CH5
- U34 pad 7: VDC -> /Feedback Channels/FB_CH6
- U34 pad 8: Net-(J24-Pad1) -> /Feedback Channels/FB_CH7
- U35 pad 1: VDC -> +3.3V
- U35 pad 2: Net-(R76-Pad1) -> GND
- U35 pad 3: Net-(R74-Pad1) -> Net-(C51-Pad1)
- U35 pad 4: GNDPWR -> Net-(C50-Pad1)
- U35 pad 5: Net-(R76-Pad1) -> Net-(TP13-Pad1)
- U35 pad 6: unconnected-(U35-Pad6) -> Net-(TP14-Pad1)
- U35 pad 7: VBUS -> VDC
- U35 pad 8: Net-(R77-Pad2) -> Net-(J23-Pad1)
- U36 pad 1: Net-(C36-Pad1) -> VDC
- U36 pad 2: GND -> Net-(R78-Pad1)
- U36 pad 3: /SCL -> Net-(R76-Pad1)
- U36 pad 4: /SDA -> GNDPWR
- U36 pad 5: +3.3V -> Net-(R78-Pad1)
- U36 pad 6: Net-(C37-Pad1) -> unconnected-(U36-Pad6)
- U37 pad 1: Net-(C41-Pad1) -> Net-(C54-Pad1)
- U37 pad 2: VBUS -> GND
- U37 pad 3: VBUS -> /SCL
- U37 pad 4: Net-(R83-Pad1) -> /SDA
- U37 pad 5: Net-(R86-Pad2) -> +3.3V
- U37 pad 6: Net-(C43-Pad1) -> Net-(C55-Pad1)
- U38 pad 1: Net-(R90-Pad2) -> Net-(C59-Pad1)
- U38 pad 2: Net-(D49-Pad1) -> VBUS
- U38 pad 3: Net-(J28-Pad1) -> VBUS
- U38 pad 4: Net-(D46-Pad1) -> Net-(R85-Pad1)
- U39 pad 1: +3.3V -> Net-(R94-Pad2)
- U39 pad 2: unconnected-(U39-Pad2) -> Net-(D49-Pad1)
- U39 pad 3: unconnected-(U39-Pad3) -> Net-(J27-Pad1)
- U39 pad 4: +5V -> Net-(D46-Pad1)

Commit message: 3D models, footprint updates, general board layout
Parts:
- added REF**: MountingHole_3.2mm_M3_DIN965_Pad, MountingHole:MountingHole_3.2mm_M3_DIN965_Pad, F.Cu at (173.6, -235.8)
- added REF**: MountingHole_3.2mm_M3_DIN965_Pad, MountingHole:MountingHole_3.2mm_M3_DIN965_Pad, F.Cu at (332.5, -237.9)
- added REF**: MountingHole_3.2mm_M3_DIN965_Pad, MountingHole:MountingHole_3.2mm_M3_DIN965_Pad, F.Cu at (177.0, -330.3)
- added REF**: MountingHole_3.2mm_M3_DIN965_Pad, MountingHole:MountingHole_3.2mm_M3_DIN965_Pad, F.Cu at (332.0, -328.8)
- J10, J11, J12, J13, J14, J15, J16, J17, J2, J3, J4, J5, J6, J7, J8, J9: footprint Connector_AMASS:AMASS_XT30U-M_1x02_P5.0mm_Vertical -> actuation:XT30U-M
- J18, J19, J20: footprint actuation:1751251 -> actuation:1935174
- J21, J22: footprint actuation:1751248 -> actuation:1935161
Other:
- board outline added: 178.3 x 111.8 mm

Commit message: arranged actuators, feedback
Parts:
- removed REF** (x4): MountingHole_3.2mm_M3_DIN965_Pad, MountingHole:MountingHole_3.2mm_M3_DIN965_Pad
- J10, J11, J12, J13, J14, J15, J16, J17, J2, J3, J4, J5, J6, J7, J8, J9: footprint actuation:XT30U-M -> Connector_AMASS:AMASS_XT30U-M_1x02_P5.0mm_Vertical
- J18, J19, J20: footprint actuation:1935174 -> actuation:1751251
- J21, J22: footprint actuation:1935161 -> actuation:1751248
- moved TP8 415.1 mm to (27.0, 134.5)
- moved C36 393.7 mm to (119.0, 108.0), turned to -90 degrees
- moved C33 389.7 mm to (106.5, 105.0), turned to -90 degrees
- moved C35 376.1 mm to (106.9, 108.0), turned to -90 degrees
- moved TP4 375.7 mm to (106.0, 116.5)
- moved TP7 372.5 mm to (114.5, 116.0)
- moved C21 371.3 mm to (165.0, 127.5)
- moved TP5 370.7 mm to (102.5, 116.5)
- moved C34 368.3 mm to (118.0, 105.0), turned to -90 degrees
- moved TP6 368.2 mm to (118.5, 116.5)
- moved TP3 364.6 mm to (184.6, 140.0)
- moved C24 360.9 mm to (171.0, 126.5)
- moved C12 354.1 mm to (218.9, 168.5), turned to 90 degrees
- moved C9 353.8 mm to (182.7, 167.0), turned to 90 degrees
- moved C11 353.1 mm to (206.5, 167.4), turned to 90 degrees
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Other:
- board outline removed
